File: ProvesXEPS/ProvesXEPS.kicad_pcb (KiCad board)
At the start: 4 copper layers, 87.6 x 90 mm, 10 parts, among them Q11 MBT2222ADW1T1, Q7 MBT2222ADW1T1, U10 1043, U11 1043, U13 1043, U14 1043, U15 BQ29702, U17 BQ29702

Commit message: Major Update
Changed the MPPT circuitry, fixed errors in 3.3V circuitry, updated pin definitions for 40 and 16 pin connectors, changed microcontroller, and updated the inhibit scheme.

What is still needed:
Proper battery protection, cell balancing, and fuel gauge
Parts:
- removed D1: 1N4151, Diode_THT:D_DO-35_SOD27_P7.62mm_Horizontal
- removed D2: 1N5819, Diode_THT:D_DO-41_SOD81_P10.16mm_Horizontal
- removed Q11, Q7: MBT2222ADW1T1, Package_TO_SOT_SMD:SOT-363_SC-70-6
- removed U10, U11, U13, U14: 1043, oresat-batteries:18650
- removed U15, U17: BQ29702, Package_SON:WSON-6_1.5x1.5mm_P0.5mm
Other:
- board outline removed
- board text removed: "For Instructional Use Only."
- board text removed: "SOLIDWORKS Educational Product."

Commit message: Footprints almost assigned
Got most of the footprints assigned
Parts:
- added C1: 10uF, Capacitor_SMD:C_0603_1608Metric, F.Cu at (82.2, 42.4)
- added C10: 4.7u, Capacitor_SMD:C_0402_1005Metric, F.Cu at (91.4, 61.6)
- added C14: 22u, Capacitor_SMD:C_0603_1608Metric, F.Cu at (38.0, 66.7)
- added C15: 10u, Capacitor_SMD:C_0603_1608Metric, F.Cu at (82.1, 61.1)
- added C16: 22u, Capacitor_SMD:C_0603_1608Metric, F.Cu at (47.0, 80.5)
- added C17: 10u, Capacitor_SMD:C_0603_1608Metric, F.Cu at (38.0, 69.2)
- added C18: 0.1u, Capacitor_SMD:C_0402_1005Metric, F.Cu at (132.3, 21.0)
- added C2: 22nF, Capacitor_SMD:C_0402_1005Metric, F.Cu at (76.3, 77.4)
- added C20: 3.3n, Capacitor_SMD:C_0402_1005Metric, F.Cu at (122.8, 31.2)
- added C21: 1u, Capacitor_SMD:C_0402_1005Metric, F.Cu at (112.9, 40.4)
- added C22: 10u, Capacitor_SMD:C_0603_1608Metric, F.Cu at (42.9, 80.5)
- added C23: 100u, Capacitor_SMD:C_0603_1608Metric, F.Cu at (42.9, 78.0)
- added C24: 330u, Capacitor_SMD:C_0603_1608Metric, F.Cu at (47.0, 78.0)
- added C25: 100uF, Capacitor_SMD:C_0603_1608Metric, F.Cu at (82.2, 44.9)
- added C26: 22u, Capacitor_SMD:C_0603_1608Metric, F.Cu at (30.3, 80.8)
- added C27: 27p, Capacitor_SMD:C_0402_1005Metric, F.Cu at (122.8, 29.3)
- added C28: 27p, Capacitor_SMD:C_0402_1005Metric, F.Cu at (109.7, 42.4)
- added C29: 100n, Capacitor_SMD:C_0402_1005Metric, F.Cu at (87.3, 64.8)
- added C3: .1u, Capacitor_SMD:C_0402_1005Metric, F.Cu at (116.7, 35.2)
- added C30: 100n, Capacitor_SMD:C_0402_1005Metric, F.Cu at (129.4, 23.0)
- added C31: 1u, Capacitor_SMD:C_0402_1005Metric, F.Cu at (126.5, 27.0)
- added C33: 100n, Capacitor_SMD:C_0402_1005Metric, F.Cu at (119.6, 33.2)
- added C34: 1u, Capacitor_SMD:C_0402_1005Metric, F.Cu at (94.3, 57.6)
- added C35: 100n, Capacitor_SMD:C_0402_1005Metric, F.Cu at (84.1, 69.3)
- added C36: 100n, Capacitor_SMD:C_0402_1005Metric, F.Cu at (97.3, 55.6)
- added C37: 100n, Capacitor_SMD:C_0402_1005Metric, F.Cu at (100.8, 51.6)
- added C38: 100n, Capacitor_SMD:C_0402_1005Metric, F.Cu at (100.5, 53.6)
- added C39: 100n, Capacitor_SMD:C_0402_1005Metric, F.Cu at (116.7, 37.2)
- added C4: .1u, Capacitor_SMD:C_0402_1005Metric, F.Cu at (94.3, 59.6)
- added C40: 100n, Capacitor_SMD:C_0402_1005Metric, F.Cu at (106.8, 47.3)
- added C41: 100n, Capacitor_SMD:C_0402_1005Metric, F.Cu at (109.7, 44.4)
- added C5: .1u, Capacitor_SMD:C_0402_1005Metric, F.Cu at (81.2, 71.1)
- added C6: .1u, Capacitor_SMD:C_0402_1005Metric, F.Cu at (73.4, 79.4)
- added C7: 2.2uF, Capacitor_SMD:C_0402_1005Metric, F.Cu at (72.9, 81.4)
- added C9: 3.3n, Capacitor_SMD:C_0402_1005Metric, F.Cu at (76.7, 75.4)
- added D1: 1SS355VM, Diode_SMD:D_SOD-323F, F.Cu at (26.2, 81.1)
- added D2: 1N5819, Diode_THT:D_DO-41_SOD81_P10.16mm_Horizontal, F.Cu at (37.9, 74.6)
- added D5: BAT54W, Package_TO_SOT_SMD:SOT-323_SC-70, F.Cu at (82.4, 39.3)
- added J1: Conn_01x10, Connector_JST:JST_EH_S10B-EH_1x10_P2.50mm_Horizontal, F.Cu at (27.6, 27.7)
- added J2: Conn_01x03, Connector_JST:JST_VH_S3P-VH_1x03_P3.96mm_Horizontal, F.Cu at (59.3, 58.0)
- added J3: Conn_01x03, Connector_JST:JST_VH_S3P-VH_1x03_P3.96mm_Horizontal, F.Cu at (59.3, 40.5)
- added J4: Conn_01x02, Connector_JST:JST_VH_S2P-VH_1x02_P3.96mm_Horizontal, F.Cu at (73.2, 40.5)
- added J5: Conn_01x02, Connector_JST:JST_VH_S2P-VH_1x02_P3.96mm_Horizontal, F.Cu at (88.9, 23.0)
- added L1: 33u, Inductor_SMD:L_0402_1005Metric, F.Cu at (52.0, 33.4)
- added L2: 2.2u, Inductor_SMD:L_0402_1005Metric, F.Cu at (91.5, 57.6)
- added L3: 20u, Inductor_SMD:L_0402_1005Metric, F.Cu at (129.5, 21.0)
- added L4: 330u, Inductor_SMD:L_0402_1005Metric, F.Cu at (106.8, 45.4)
- added Q10: IRLL024NTRPBF, IRLL024NTRPBF:SOT230P700X180-4N, F.Cu at (75.0, 70.3)
- added Q11: NTF5P03T3G, NTF5P03T3G:NTF5P03T3G, F.Cu at (30.9, 38.3)
- added Q12: IRLL024NTRPBF, IRLL024NTRPBF:SOT230P700X180-4N, F.Cu at (64.3, 76.5)
- added Q13: NTF5P03T3G, NTF5P03T3G:NTF5P03T3G, F.Cu at (47.0, 62.9)
- added Q14: Si2319CDS, Package_TO_SOT_SMD:SOT-23, F.Cu at (38.5, 79.0)
- added Q15: IRLL024NTRPBF, IRLL024NTRPBF:SOT230P700X180-4N, F.Cu at (54.7, 76.6)
- added Q16: IRLL024NTRPBF, IRLL024NTRPBF:SOT230P700X180-4N, F.Cu at (100.5, 46.5)
- added Q17: MMBT2222AT, MMBT2222AT:MMBT2222ATT1G, F.Cu at (84.4, 55.5)
- added Q18: MMBT2222AT, MMBT2222AT:MMBT2222ATT1G, F.Cu at (90.2, 44.3)
- added Q21: NTF5P03T3G, NTF5P03T3G:NTF5P03T3G, F.Cu at (60.4, 27.9)
- added Q22: Q_NPN_CEB, MMBT2222AT:MMBT2222ATT1G, F.Cu at (100.1, 26.9)
- added Q23: Q_NPN_CEB, MMBT2222AT:MMBT2222ATT1G, F.Cu at (100.1, 38.1)
- added Q24: Q_NPN_CEB, MMBT2222AT:MMBT2222ATT1G, F.Cu at (74.5, 61.8)
- added Q25: Q_NPN_CEB, MMBT2222AT:MMBT2222ATT1G, F.Cu at (110.0, 26.9)
- added Q5: NTF5P03T3G, NTF5P03T3G:NTF5P03T3G, F.Cu at (47.0, 45.4)
- added Q6: IRLL024NTRPBF, IRLL024NTRPBF:SOT230P700X180-4N, F.Cu at (120.3, 24.1)
- added Q7: IRLL024NTRPBF, IRLL024NTRPBF:SOT230P700X180-4N, F.Cu at (110.5, 35.3)
- added Q8: NTF5P03T3G, NTF5P03T3G:NTF5P03T3G, F.Cu at (30.9, 55.8)
- added Q9: NTF5P03T3G, NTF5P03T3G:NTF5P03T3G, F.Cu at (76.6, 27.9)
- added R1: 100, Resistor_SMD:R_0402_1005Metric, F.Cu at (88.5, 60.8)
- added R11: 715k, Resistor_SMD:R_0402_1005Metric, F.Cu at (91.5, 59.6)
- added R13: 102k, Resistor_SMD:R_0402_1005Metric, F.Cu at (106.8, 43.4)
- added R17: 10k, Resistor_SMD:R_0402_1005Metric, F.Cu at (116.7, 33.2)
- added R19: 845k, Resistor_SMD:R_0402_1005Metric, F.Cu at (119.9, 31.3)
- added R2: 0.1, Resistor_SMD:R_0402_1005Metric, F.Cu at (73.8, 75.4)
- added R20: 3.01k, Resistor_SMD:R_0402_1005Metric, F.Cu at (126.5, 21.0)
- added R21: 2.1M, Resistor_SMD:R_0402_1005Metric, F.Cu at (126.5, 25.0)
- added R23: 100k, Resistor_SMD:R_0402_1005Metric_Pad0.72x0.64mm_HandSolder, F.Cu at (91.6, 51.6)
- added R25: 107k, Resistor_SMD:R_0402_1005Metric, F.Cu at (94.7, 53.6)
- added R27: 100k, Resistor_SMD:R_0402_1005Metric_Pad0.72x0.64mm_HandSolder, F.Cu at (81.8, 47.2)
- added R28: 470k, Resistor_SMD:R_0402_1005Metric, F.Cu at (126.5, 23.0)
- added R3: 1k, Resistor_SMD:R_0402_1005Metric, F.Cu at (87.4, 62.8)
- added R30: 100k, Resistor_SMD:R_0402_1005Metric_Pad0.72x0.64mm_HandSolder, F.Cu at (33.9, 80.6)
- added R31: 100k, Resistor_SMD:R_0402_1005Metric_Pad0.72x0.64mm_HandSolder, F.Cu at (61.1, 81.7)
- added R32: 470k, Resistor_SMD:R_0402_1005Metric, F.Cu at (81.2, 67.1)
- added R34: 73.2k, Resistor_SMD:R_0402_1005Metric, F.Cu at (110.0, 40.4)
- added R35: 22.1k, Resistor_SMD:R_0402_1005Metric, F.Cu at (70.0, 81.7)
- added R36: 100k, Resistor_SMD:R_0402_1005Metric, F.Cu at (84.2, 67.3)
- added R37: 10k, Resistor_SMD:R_0402_1005Metric, F.Cu at (117.0, 29.3)
- added R38: 10k, Resistor_SMD:R_0402_1005Metric, F.Cu at (52.0, 35.4)
- added R39: 20k, Resistor_SMD:R_0402_1005Metric, F.Cu at (97.6, 53.6)
- added R4: 100, Resistor_SMD:R_0402_1005Metric, F.Cu at (81.2, 69.1)
- added R40: 20k, Resistor_SMD:R_0402_1005Metric, F.Cu at (117.0, 31.3)
- added R41: 10k, Resistor_SMD:R_0402_1005Metric, F.Cu at (64.2, 81.7)
- added R42: 10k, Resistor_SMD:R_0402_1005Metric, F.Cu at (98.0, 51.6)
- added R43: 10k, Resistor_SMD:R_0402_1005Metric, F.Cu at (91.5, 55.6)
- added R44: 107k, Resistor_SMD:R_0402_1005Metric, F.Cu at (67.1, 81.7)
- added R45: 10k, Resistor_SMD:R_0402_1005Metric, F.Cu at (94.4, 55.6)
- added R46: 10k, Resistor_SMD:R_0402_1005Metric, F.Cu at (70.5, 77.4)
- added R47: 10k, Resistor_SMD:R_0402_1005Metric, F.Cu at (70.5, 79.4)
- added R48: 4.7k, Resistor_SMD:R_0402_1005Metric, F.Cu at (73.4, 77.4)
- added R49: 4.7k, Resistor_SMD:R_0402_1005Metric, F.Cu at (107.1, 40.4)
- added R5: 536k, Resistor_SMD:R_0402_1005Metric, F.Cu at (84.2, 65.3)
- added R50: 100k, Resistor_SMD:R_0402_1005Metric, F.Cu at (85.6, 60.8)
- added R51: 100k, Resistor_SMD:R_0402_1005Metric, F.Cu at (52.0, 31.4)
- added R52: 1k, Resistor_SMD:R_0402_1005Metric, F.Cu at (119.9, 29.3)
- added R55: 1k, Resistor_SMD:R_0402_1005Metric_Pad0.72x0.64mm_HandSolder, F.Cu at (70.7, 75.4)
- added R56: 27, Resistor_SMD:R_0402_1005Metric_Pad0.72x0.64mm_HandSolder, F.Cu at (91.6, 49.6)
- added R57: 27, Resistor_SMD:R_0402_1005Metric_Pad0.72x0.64mm_HandSolder, F.Cu at (91.6, 53.6)
- added R58: DNF, Resistor_SMD:R_0402_1005Metric_Pad0.72x0.64mm_HandSolder, F.Cu at (94.9, 51.6)
- added R6: 100k, Resistor_SMD:R_0402_1005Metric_Pad0.72x0.64mm_HandSolder, F.Cu at (37.7, 71.4)
- added R7: 1k, Resistor_SMD:R_0402_1005Metric, F.Cu at (81.5, 63.3)
- added R8: 1k, Resistor_SMD:R_0402_1005Metric, F.Cu at (84.5, 63.3)
- added U16: W25Q128JVS, Package_SO:SOIC-8_5.23x5.23mm_P1.27mm, F.Cu at (45.4, 33.8)
- added U2: BQ28400PWR, BQ28400PWR:BQ28400PWR, F.Cu at (30.3, 73.4)
