File: ProvesXEPS/ProvesXEPS.kicad_sch (KiCad schematic)
At the start: 143 parts, among them IC1 PIC18F16Q41-E_SS, IC2 S-8209AAC-T8T1U, IC3 S-8209AAC-T8T1U, IC4 LTC4121, IC5 PCA9543AD, IC6 TPS54226PWPR, J1 Conn_01x10, J2 Conn_01x03, J3 Conn_01x03, J4 M50-3900842, J5 M50-3902042, K1 PE014006, K2 PE014006, Q1 PMV45EN2R, Q10 IRLL024NTRPBF, Q11 MBT2222ADW1T1, Q12 NTF6P02T3G, Q13 NTF6P02T3G, Q14 IRLL024NTRPBF, Q15 IRLL024NTRPBF, Q16 NTF6P02T3G, Q17 MMBT2222AT, Q18 MMBT2222AT, Q19 IRLML2803TRPBF, Q2 PMV45EN2R, Q20 IRLML2803TRPBF, Q21 NDS8434, Q22 NDS8434, Q3 PMV45EN2R, Q4 PMV45EN2R, Q5 IRLL024NTRPBF, Q6 IRLL024NTRPBF, Q7 MBT2222ADW1T1, Q8 NTF6P02T3G, Q9 NTF6P02T3G, U1 ADM1176-1ARMZ-R7, U10 1043, U11 1043, U12 IRF7503TRPBF, U13 1043, U14 1043, U15 BQ29702, U16 IRF7503TRPBF, U17 BQ29702, U2 LTC4412ES6-TRPBF, U3 SI7625DN-T1-GE3, U4 SI7625DN-T1-GE3, U5 MAX17205G+T, U6 SI7625DN-T1-GE3, U7 SI7625DN-T1-GE3, U8 LTC4412ES6-TRPBF, U9 TL2575HV-05QKTTRQ1

Commit message: Schematic Update
Added crystal. changed a couple of nets, and added stuff we still need to do
Parts:
- removed R6: 1k, symbol Device:R_US
- added C? (x2): 3.9p, symbol Device:C
- added R?: 47k, symbol Device:R_US
- added Y?: 32kHz, microchip_osc:VMK3-9001-32K7680000, symbol Device:Crystal
- R23, R25, R28, R30, R31, R32: value 470 -> 4k7
- U10: footprint (none) -> oresat-batteries:18650
Connections:
- net +3V3: now also IC1.1 (VDD), R?.2
- net EN_Burn1: now also IC1.18 (RA1/ICSPCLK); no longer IC1.2 (RA5)
- net EN_Burn2: now also IC1.16 (RC0); no longer IC1.3 (RA4)
- net GND: now also C?.2, C?.2; no longer IC4.6 (MPPT), R11.2, R13.1
- net GPIO11: no longer IC1.16 (RC0)
- net VBat_Pos: no longer C25.1, U9.1 (VIN)
- net VBatt: no longer C15.1, C17.1, IC1.1 (VDD), IC6.13 (VIN), IC6.14 (VCC)
- net at S1.2: now also IC1.4 (~{MCLR}/VPP/RA3), R?.1
- net PwrMon renamed Inhb_o
- net Inhb_o: now also C15.1, C17.1, C25.1, IC6.13 (VIN), IC6.14 (VCC), U9.1 (VIN)
- new net: IC4.6 (MPPT), R11.2, R13.1
- new net osc_i: C?.1, IC1.2 (RA5), Y?.1
- new net osc_o: C?.1, IC1.3 (RA4), Y?.2
- no-connect marks 67 -> 66
Other:
- note added: "Still need: - number label components - reassign footprints - Debugger Circuit for pic - Examine Power monitor input"
- note added: "VMK3-9001-32K7680000TR"
- note added: "crystal"
- note removed: "Still need: - number label components - reassign footprints"

Commit message: Major Update
Changed the MPPT circuitry, fixed errors in 3.3V circuitry, updated pin definitions for 40 and 16 pin connectors, changed microcontroller, and updated the inhibit scheme.

What is still needed:
Proper battery protection, cell balancing, and fuel gauge
Parts:
- removed C? (x2): 3.9p, symbol Device:C
- removed IC1: PIC18F16Q41-E_SS, SOP65P780X200-20N, symbol PIC18F16Q41-E_SS:PIC18F16Q41-E_SS
- removed IC5: PCA9543AD, SOIC127P600X175-14N, symbol PCA9543AD:PCA9543AD
- removed J4: M50-3900842, M50-3900842, symbol M50-3900842:M50-3900842
- removed J5: M50-3902042, M50-3902042, symbol M50-3902042:M50-3902042
- removed Q11, Q7: MBT2222ADW1T1, Package_TO_SOT_SMD:SOT-363_SC-70-6, symbol Transistor_BJT:MBT2222ADW1T1
- removed Q12, Q16: NTF6P02T3G, SOT230P700X175-4N, symbol NTF6P02T3G:NTF6P02T3G
- removed Q14, Q5: IRLL024NTRPBF, SOT230P700X180-4N, symbol IRLL024NTRPBF:IRLL024NTRPBF
- removed Q21, Q22: NDS8434, SOIC127P600X175-8N, symbol NDS8434:NDS8434
- removed R44: 0.01, symbol Device:R
- removed R?: 47k, symbol Device:R_US
- removed S1: GPTS203211B, digikey-footprints:PushButton_12x12mm_THT_GPTS203211B, symbol dk_Pushbutton-Switches:GPTS203211B
- removed U12, U16: IRF7503TRPBF, IRF7503TRPBF_INF, symbol Imported_Symbols:IRF7503TRPBF
- removed Y?: 32kHz, microchip_osc:VMK3-9001-32K7680000, symbol Device:Crystal
- added C26: 22u, symbol Device:C
- added C27, C28: 27p, Capacitor_SMD:C_0402_1005Metric, symbol Device:C
- added C29, C30, C33, C35, C36, C37, C38, C39, C40, C41: 100n, Capacitor_SMD:C_0402_1005Metric, symbol Device:C
- added C31, C34: 1u, Capacitor_SMD:C_0402_1005Metric, symbol Device:C
- added C32: .1u, Capacitor_SMD:C_0402_1005Metric, symbol Device:C
- added D5: BAT54W, Package_TO_SOT_SMD:SOT-323_SC-70, symbol Diode:BAT54W
- added J4: Conn_01x02, symbol Connector_Generic:Conn_01x02
- added J5: Conn_01x02, Connector_PinHeader_2.54mm:PinHeader_1x02_P2.54mm_Vertical, symbol Connector_Generic:Conn_01x02
- added J6: USB_B_Micro, RP2040_minimal:USB_Micro-B_Amphenol_10103594-0001LF_Horizontal_modified, symbol RP2040_minimal-rescue:USB_B_Micro-Connector
- added J7: M50-3902042, SamacSys_Parts:M50-3902042, symbol SamacSys_Parts:M50-3902042
- added J8: M50-3900842, symbol M50-3900842:M50-3900842
- added Q11, Q21, Q5: NTF5P03T3G, NTF5P03T3G:NTF5P03T3G, symbol NTF6P02T3G:NTF6P02T3G
- added Q12, Q16, Q7: IRLL024NTRPBF, IRLL024NTRPBF:SOT230P700X180-4N, symbol IRLL024NTRPBF:IRLL024NTRPBF
- added Q14: Si2319CDS, Package_TO_SOT_SMD:SOT-23, symbol Transistor_FET:Si2319CDS
- added Q22, Q23, Q24, Q25: Q_NPN_CEB, MMBT2222AT:MMBT2222ATT1G, symbol Device:Q_NPN_CEB
- added Q26, Q27: IRF7404, SOIC127P600X175-8N, symbol IRF7404:IRF7404
- added R44: 107k, symbol Device:R_US
- added R52, R55: 1k, Capacitor_SMD:C_0402_1005Metric, symbol Device:R
- added R53: 330, Resistor_SMD:R_0402_1005Metric_Pad0.72x0.64mm_HandSolder, symbol Device:R_US
- added R54, R59: 2.2k, Resistor_SMD:R_0402_1005Metric_Pad0.72x0.64mm_HandSolder, symbol Device:R_US
- added R56, R57: 27, Capacitor_SMD:C_0402_1005Metric, symbol Device:R
- added R58: DNF, Capacitor_SMD:C_0402_1005Metric, symbol Device:R
- added R6: 100k, Resistor_SMD:R_0402_1005Metric_Pad0.72x0.64mm_HandSolder, symbol Device:R_US
- added U12: RP2040, RP2040_minimal:RP2040-QFN-56, symbol MCU_RaspberryPi_RP2040:RP2040
- added U16: W25Q128JVS, Package_SO:SOIC-8_5.23x5.23mm_P1.27mm, symbol Memory_Flash:W25Q128JVS
- added Y1: ABLS-12.000MHZ-B4-T, RP2040_minimal:Crystal_SMD_HC49-US, symbol Device:Crystal
- C10: value 22u -> 4.7u
- C15, C17: value 100u -> 10u
- J1: footprint (none) -> Connector_JST:JST_EH_S10B-EH_1x10_P2.50mm_Horizontal
- L1: value 33uH -> 33u
- L2: value 3.3u -> 2.2u
- Q10, Q15, Q6: footprint SOT230P700X180-4N -> IRLL024NTRPBF:SOT230P700X180-4N
- Q13, Q8, Q9: value NTF6P02T3G -> NTF5P03T3G; footprint SOT230P700X175-4N -> NTF5P03T3G:NTF5P03T3G
- Q17, Q18: footprint SOTFL50P160X78-3N -> MMBT2222AT:MMBT2222ATT1G
- R11: value 787k -> 715k
- R13: value 121k -> 102k
- R17: value 100k -> 10k
- R23, R30, R31: value 4k7 -> 100k; footprint (none) -> Resistor_SMD:R_0402_1005Metric_Pad0.72x0.64mm_HandSolder
- R25: value 4k7 -> 107k
- R27: value 470 -> 100k; footprint (none) -> Resistor_SMD:R_0402_1005Metric_Pad0.72x0.64mm_HandSolder
- R28, R32: value 4k7 -> 470k
- R5: value 0 -> 536k
Connections:
- net I2C2_SCL is gone; now on net GND: R30.2
- net I2C2_SDA is gone; now on net VBatt: R32.2
- net VBat_Pos is gone; now on net VBatt: U13.2, U14.2, U17.5 (BAT)
- net +3V3: now also C39.1, R58.1, U16.8 (VCC); no longer IC4.15 (~{FAULT}), R17.2, R23.2, R25.2, R27.2, R28.1, R30.1, R31.1, R32.1
- net +5V: now also J7.1, J7.2
- net BurnRelay1: now also U12.16 (GPIO13)
- net BurnRelay2: now also U12.17 (GPIO14)
- net EN_Burn1: now also U12.14 (GPIO11)
- net EN_Burn2: now also U12.15 (GPIO12)
- net F1: now also Q6.1 (GATE), Q9.1 (G), R27.1; no longer Q8.1 (G)
- net F2: now also R30.1, Q11.1 (G), Q12.1 (GATE); no longer Q13.1 (G), Q6.1 (GATE)
- net F3: now also Q6.3 (SOURCE), Q8.1 (G), R23.1, Q7.1 (GATE); no longer Q9.1 (G)
- net F4: now also Q10.1 (GATE), Q13.1 (G), Q13.2 (D_1), Q8.2 (D_1), R31.1, Q12.3 (SOURCE), Q5.3 (S); no longer Q15.1 (GATE)
- net GND: now also Q10.3 (SOURCE), Q15.3 (SOURCE), R17.1, R23.2, R27.2, R31.2, C26.2, C27.2, C28.2, C29.2, C30.2, C31.2, C33.2, C34.2, C35.2, C36.2, C37.2, C38.2, C39.2, C40.2, C41.2, J5.2 (Pin_2), J6.5 (GND), J6.6 (Shield), J7.11, J7.17, J7.19, J7.26, J7.3, J7.35, J7.36, J7.37, J7.39, J7.4, J7.7, J7.8, J7.9, J8.13, J8.14, J8.5, Q16.3 (SOURCE), Q22.2 (E), Q23.2 (E), Q24.2 (E), Q25.2 (E), Q7.3 (SOURCE), R54.2, R6.2, U12.19 (TESTEN), U12.57 (GND), U16.4 (GND); no longer C7.1, IC4.7 (FREQ), Q13.2 (D_1), Q8.2 (D_1), Q9.2 (D_1)
- net RBF: now also Q15.1 (GATE), Q5.1 (G), R6.1; no longer Q10.1 (GATE)
- net SCL_I2C_1: now also U12.9 (GPIO7); no longer R31.2
- net SDA_I2C_1: now also U12.8 (GPIO6); no longer R28.2
- net VBUS_RESET: now also U12.13 (GPIO10)
- net VBatt: now also Q9.3 (S), C26.1, J8.3, J8.4, Q11.3 (S), Q14.2 (S), Q21.3 (S), R44.1; no longer C10.1, IC4.9 (BAT), R21.2
- net VSolar: now also D5.1 (A), J8.1, J8.2; no longer C1.1, C2.2, IC4.3 (IN), IC4.4 (SW), J2.2 (Pin_2), J3.2 (Pin_2), L1.2, R11.1, R5.1
- net at C22.2, R41.2: now also Q24.1 (C), Q25.1 (C)
- net at R42.1: now also Q25.3 (B)
- net at C22.1, R40.1: now also Q23.3 (B)
- net at IC4.16 (RUN), R5.2: now also R25.2
- net SCL_I2C_0: now reaches U1.6 (SCL)
- net SCL_I2C_0: now also U12.12 (GPIO9); no longer R23.1
- net at R25.1: now also C7.1, R17.2; no longer U1.7 (SDA)
- net at Q19.3, R50.2: now also Q27.4
- net at C7.2, IC4.1 (INTVCC): now also IC4.7 (FREQ)
- net at IC4.14 (~{CHRG}): now also Q14.1 (G), R44.2; no longer R17.1
- net at K1.2 (11_COM), R51.1: now also Q26.1, Q26.2, Q26.3
- net at Q20.3, R51.2: now also Q26.4
- net at J3.3 (Pin_3): now also Q26.5, Q26.6, Q26.7, Q26.8
- net at R38.2, R39.1: now also Q22.3 (B), Q23.1 (C)
- net at K2.2 (11_COM), R50.1: now also Q27.1, Q27.2, Q27.3
- net at IC6.7 (EN), R37.2: now also Q22.1 (C)
- net at R39.2: now also Q24.3 (B)
- net at J2.3 (Pin_3): now also Q27.5, Q27.6, Q27.7, Q27.8
- net at Q15.2 (DRAIN_1): now also Q6.2 (DRAIN_1), Q12.2 (DRAIN_1), Q16.1 (GATE), Q21.1 (G), Q5.2 (D_1)
- net Inhb_o renamed inhibit_out
- net inhibit_out: now also Q16.2 (DRAIN_1), Q21.2 (D_1); no longer Q10.3 (SOURCE), Q13.3 (S), Q8.3 (S)
- net VBat_Mid renamed pack + (1)
- net pack + (1): now also R53.1; no longer U15.5 (BAT), U17.4 (VSS), U17.6 (V-)
- net VBat_Neg: no longer names the net of U10.1, U11.1
- net VBat_Neg: now also C32.2; no longer U15.4 (VSS), U15.6 (V-)
- new net: Q11.2 (D_1), Q13.3 (S), Q8.3 (S), Q9.2 (D_1)
- new net: C1.1, D5.3 (K), IC4.3 (IN), R11.1, R28.1, R5.1
- new net: C28.1, R52.2, Y1.2
- new net: IC4.15 (~{FAULT}), R28.2
- new net: C2.2, IC4.4 (SW), L1.2
- new net: C10.1, IC4.9 (BAT), Q14.3 (D), R21.2, R32.1
- new net: R57.2, U12.46 (USB_DM)
- new net: R59.1, U17.6 (V-)
- new net: R54.1, U15.6 (V-)
- new net: C32.1, R53.2, U15.5 (BAT)
- new net: R56.2, U12.47 (USB_DP)
- new net +1V1: C29.1, C30.1, C31.1, U12.23 (DVDD), U12.45 (VREG_VOUT), U12.50 (DVDD)
- new net +3.3V: C33.1, C34.1, C35.1, C36.1, C37.1, C38.1, C40.1, C41.1, J7.5, J7.6, J8.6, U12.1 (IOVDD), U12.10 (IOVDD), U12.22 (IOVDD), U12.26 (RUN), U12.33 (IOVDD), U12.42 (IOVDD), U12.43 (ADC_AVDD), U12.44 (VREG_IN), U12.48 (USB_VDD), U12.49 (IOVDD)
- new net Burn WIre: J3.2 (Pin_2)
- new net GPIO5: J7.18, U12.18 (GPIO15)
- new net Heat Pad: J2.2 (Pin_2)
- new net QSPI_SCLK: U12.52 (QSPI_SCLK), U16.6 (CLK)
- new net QSPI_SD0: U12.53 (QSPI_SD0), U16.5 (DI(IO0))
- new net QSPI_SD1: U12.55 (QSPI_SD1), U16.2 (DO(IO1))
- new net QSPI_SD2: U12.54 (QSPI_SD2), U16.3 (IO2)
- new net QSPI_SD3: U12.51 (QSPI_SD3), U16.7 (IO3)
- new net QSPI_SS: R55.1, R58.2, U12.56 (QSPI_SS), U16.1 (~{CS})
- new net SDA_I2C_0: U1.7 (SDA), U12.11 (GPIO8)
- new net SPIO_CS: J7.34, U12.7 (GPIO5)
- new net SPIO_MISO: J7.32, U12.6 (GPIO4)
- new net SPIO_MOSI: J7.30, U12.5 (GPIO3)
- new net SPIO_SCK: J7.28, U12.4 (GPIO2)
- new net SWCLK: J4.2 (Pin_2), U12.24 (SWCLK)
- new net SWD: J4.1 (Pin_1), U12.25 (SWD)
- new net UART0_RX: J7.38, U12.3 (GPIO1)
- new net UART0_TX: J7.40, U12.2 (GPIO0)
- new net USB_D+: J6.3 (D+), R56.1
- new net USB_D-: J6.2 (D-), R57.1
- new net XIN: C27.1, U12.20 (XIN), Y1.1
- new net XOUT: R52.1, U12.21 (XOUT)
- new net ~{USB_BOOT}: J5.1 (Pin_1), R55.2
- now unconnected: Q10.2 (DRAIN_1)
- no-connect marks 66 -> 78
Other:
- note added: "Burn Wire"
- note added: "Flash"
- note added: "Make sure C10 is close to pin 44 of RP2040"
- note added: "Make sure C8 is close to pin 45 of RP2040"
- note added: "Make sure R3 and R4 are close to RP2040"
- note added: "Relay Circuitry"
- note removed: "Burn Relay"
- note removed: "Fuel Gauge"
- note removed: "I2C MUX"
- note removed: "MCU"
- note removed: "OV/UV Protection (4.6V/2.8V) OCD/SCD Protection (3.5A OCD)"
- note removed: "SPI Clock Slave Select"
- note removed: "Still need: - number label components - reassign footprints - Debugger Circuit for pic - Examine Power monitor input"
- note removed: "VMK3-9001-32K7680000TR"
- moved on the sheet: C1, C9, R2, R3, R5, U1

Commit message: Change to protection circuitry
Parts:
- removed C11, C19: 100n, symbol Device:C
- removed C12, C13: 470n, symbol Device:C
- removed C32: .1u, Capacitor_SMD:C_0402_1005Metric, symbol Device:C
- removed C8: 10n, symbol Device:C
- removed D1: 1N4151, Diode_THT:D_DO-35_SOD27_P7.62mm_Horizontal, symbol Diode:1N4151
- removed F1: 1206L500_12SLPR, 1206L075SLYR, symbol 1206L500/12SLPR:1206L500_12SLPR
- removed F2: 1206L150_12SLYR, 1206L075SLYR, symbol 1206L150/12SLYR:1206L150_12SLYR
- removed IC2, IC3: S-8209AAC-T8T1U, SOP65P640X110-8N, symbol S-8209AAC-T8T1U:S-8209AAC-T8T1U
- removed Q1, Q2, Q3, Q4: PMV45EN2R, SOT95P230X110-3N, symbol PMV45EN2R:PMV45EN2R
- removed R10: 470, symbol Device:R_US
- removed R12, R14, R18, R26, R9: 100k, symbol Device:R_US
- removed R15, R16: 1k, symbol Device:R_US
- removed R22: 10, symbol Device:R_US
- removed R24: 10m, symbol Device:R_US
- removed R29, R33: 10k, symbol Device:R_US
- removed R53: 330, Resistor_SMD:R_0402_1005Metric_Pad0.72x0.64mm_HandSolder, symbol Device:R_US
- removed R54, R59: 2.2k, Resistor_SMD:R_0402_1005Metric_Pad0.72x0.64mm_HandSolder, symbol Device:R_US
- removed TH1, TH2: Thermistor_NTC, symbol Device:Thermistor_NTC
- removed TP1: Discharge Stat, symbol Connector:TestPoint
- removed TP2: Charge Stat, symbol Connector:TestPoint
- removed U15, U17: BQ29702, Package_SON:WSON-6_1.5x1.5mm_P0.5mm, symbol Battery_Management:BQ297xy
- removed U2, U8: LTC4412ES6-TRPBF, LTC4412ES6-TRPBF_ADI, symbol LTC4412ES6#TRPBF:LTC4412ES6-TRPBF
- removed U3, U4, U6, U7: SI7625DN-T1-GE3, MOSFET_1DN-T1-GE3_VIS, symbol SI7625DN-T1-GE3:SI7625DN-T1-GE3
- removed U5: MAX17205G+T, 21-0137_T1433-2C_MXM, symbol 2022-03-31_06-47-44:MAX17205G+T
- added D1: 1SS355VM, Diode_SMD:D_SOD-323F, symbol Diode:1SS355VM
- added U2: BQ28400PWR, BQ28400PWR:BQ28400PWR, symbol BQ28400PWR:BQ28400PWR
- C1, C14, C15, C16, C17, C22, C23, C24, C25, C26: footprint (none) -> Capacitor_SMD:C_0603_1608Metric
- C10, C18, C2, C20, C21, C7, C9: footprint (none) -> Capacitor_SMD:C_0402_1005Metric
- C3, C4, C6: value 100n -> .1u; footprint (none) -> Capacitor_SMD:C_0402_1005Metric
- C5: value 10n -> .1u; footprint (none) -> Capacitor_SMD:C_0402_1005Metric
- J2, J3: footprint (none) -> Connector_JST:JST_VH_S3P-VH_1x03_P3.96mm_Horizontal
- J4: footprint (none) -> Connector_JST:JST_VH_S2P-VH_1x02_P3.96mm_Horizontal
- J5: footprint Connector_PinHeader_2.54mm:PinHeader_1x02_P2.54mm_Vertical -> Connector_JST:JST_VH_S2P-VH_1x02_P3.96mm_Horizontal
- J7: footprint SamacSys_Parts:M50-3902042 -> (none)
- R1: value 1k -> 100
- R4: value 100k -> 100
- R7: value 470 -> 1k
Connections:
- net GND: now also C3.2, C6.2, U10.1, U11.1, U2.15 (VSS)
- net SCL_I2C_1: now also U2.10 (SMBD), U2.12 (SMBC)
- net VBatt: now also R4.1, D1.2 (A), U2.2 (DSG); no longer C26.1, Q14.2 (S), R32.2, R44.1, U13.2, U14.2
- net at C5.2: now also C3.1, R1.2, U2.6 (SRP); no longer C3.2
- net at R8.2: now also U2.4 (VC2)
- net at C4.1: now also C5.1, R4.2, U2.7 (SRN)
- net Batt2+: now reaches R1.1
- net Batt2+: now also R7.1
- net at C6.1: now also U2.14 (RBI)
- net pack + (1) renamed batt1+
- new net: R7.2, U2.3 (VC1)
- new net: D1.1 (K), U2.20 (PACK)
- new net Batt1+: R8.1
- new net Batt1-: U2.5 (VSS)
- new net VCHG: C26.1, Q14.2 (S), R32.2, R44.1, U2.19 (CHG)
- new net batt2+: U13.2, U14.2
- no-connect marks 78 -> 61
Other:
- note removed: "Charge Protection"
- note removed: "Charge Switch"
- note removed: "Discharge Switch"
- note removed: "Fuel Gauge & Cell Balancing"
- note removed: "Honeywell 197-103LAG-A01"
- note removed: "Power Path 1"
- moved on the sheet: U10, U11, U13, U14

Commit message: Footprints almost assigned
Got most of the footprints assigned
Parts:
- D3, D4: footprint POWERDI_123 -> (none)
- IC4: footprint QFN50P300X300X80-17N-D -> (none)
- IC6: footprint SOP65P640X120-15N -> (none)
- J6: footprint RP2040_minimal:USB_Micro-B_Amphenol_10103594-0001LF_Horizontal_modified -> (none)
- K1, K2: footprint 1415390-1 -> (none)
- L1, L2, L3, L4: footprint (none) -> Inductor_SMD:L_0402_1005Metric
- Q19, Q20: footprint SOT95P237X112-3N -> (none)
- Q26, Q27: footprint SOIC127P600X175-8N -> (none)
- R1, R11, R13, R17, R19, R2, R20, R21, R25, R28, R3, R32, R34, R35, R36, R37, R38, R39, R4, R40, R41, R42, R43, R44, R45, R46, R47, R48, R49, R5, R50, R51, R7, R8: footprint (none) -> Resistor_SMD:R_0402_1005Metric
- R52: footprint Capacitor_SMD:C_0402_1005Metric -> Resistor_SMD:R_0402_1005Metric
- R55, R56, R57, R58: footprint Capacitor_SMD:C_0402_1005Metric -> Resistor_SMD:R_0402_1005Metric_Pad0.72x0.64mm_HandSolder
- U1: footprint RM_10_ADI -> (none)
- U10, U11, U13, U14: footprint oresat-batteries:18650 -> (none)
- U12: footprint RP2040_minimal:RP2040-QFN-56 -> (none)
- U9: footprint KTT5 -> (none)
- Y1: footprint RP2040_minimal:Crystal_SMD_HC49-US -> (none)
